Commit message: Add files via upload

File: pioneer_description/urdf/PruebaCopelia.urdf (robot description, URDF)
Before this commit: robot Pioneer_2-AT_8, 13 links, 12 joints
Links:
- link Eje_der_delantero_link: geometry collision mesh filename=/home/victorguti/catkin_ws/src/pioneer_description/meshes/e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; visual mesh filename=/home/victorguti/catkin_ws/src/pioneer_description/meshes/e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
- link Eje_der_trasero_link: geometry collision mesh filename=/home/victorguti/catkin_ws/src/pioneer_description/meshes/e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; visual mesh filename=/home/victorguti/catkin_ws/src/pioneer_description/meshes/e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
- link Eje_izq_delantero_link: geometry collision mesh filename=/home/victorguti/catkin_ws/src/pioneer_description/meshes/e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; visual mesh filename=/home/victorguti/catkin_ws/src/pioneer_description/meshes/e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
- link Eje_izq_trasero_link: geometry collision mesh filename=/home/victorguti/catkin_ws/src/pioneer_description/meshes/e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; visual mesh filename=/home/victorguti/catkin_ws/src/pioneer_description/meshes/e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
- link Rueda_der_delantera_link: geometry collision cylinder length=0.075 radius=0.111; visual mesh filename=/home/victorguti/catkin_ws/src/pioneer_description/meshes/r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
- link Rueda_der_trasera_link: geometry collision cylinder length=0.075 radius=0.111; visual mesh filename=/home/victorguti/catkin_ws/src/pioneer_description/meshes/r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
- link Rueda_izq_delantera_link: geometry collision cylinder length=0.075 radius=0.111; visual mesh filename=/home/victorguti/catkin_ws/src/pioneer_description/meshes/r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
- link Rueda_izq_trasera_link: geometry collision cylinder length=0.075 radius=0.111; visual mesh filename=/home/victorguti/catkin_ws/src/pioneer_description/meshes/r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
- link Sonar_delantero_link: geometry collision mesh filename=/home/victorguti/catkin_ws/src/pioneer_description/meshes/s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; visual mesh filename=/home/victorguti/catkin_ws/src/pioneer_description/meshes/s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
- link Sonar_trasero_link: geometry collision mesh filename=/home/victorguti/catkin_ws/src/pioneer_description/meshes/s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; visual mesh filename=/home/victorguti/catkin_ws/src/pioneer_description/meshes/s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
- link base_link: geometry collision mesh filename=/home/victorguti/catkin_ws/src/pioneer_description/meshes/c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; visual mesh filename=/home/victorguti/catkin_ws/src/pioneer_description/meshes/c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
- link cubierta_link: geometry collision mesh filename=/home/victorguti/catkin_ws/src/pioneer_description/meshes/c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; visual mesh filename=/home/victorguti/catkin_ws/src/pioneer_description/meshes/c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

File: pioneer_description/urdf/pioneer_lidar.urdf (robot description, URDF)
Before this commit: robot Pioneer_2-AT_8, 13 links, 12 joints
Links:
- removed link lidar_link
- added link hokuyo_link, mass 1e-5; collision mesh filename=package://pioneer_description/meshes/hokuyo.dae; visual mesh filename=package://pioneer_description/meshes/hokuyo.dae
- link base_link: geometry collision box size=0.5 0.38 0.19; visual mesh filename=package://pioneer_description/meshes/chasis.stl
- link cubierta_link: geometry collision box size=0.51 0.38 0.03; visual mesh filename=package://pioneer_description/meshes/cubierta.stl
Joints:
- removed joint lidar_cubierta
- added joint hokuyo_joint: type fixed, parent base_link, child hokuyo_link, origin xyz=0.136 0 0.309 rpy=0 0 0, axis 0 1 0
