Commit message: pre foxy

File: src/description/gazebo_control.xacro (robot description, xacro)
@@ -7,5 +7,5 @@
             <right_joint>base_ruedaderdel_joint</right_joint>
             <wheel_separation>0.415</wheel_separation>
-            <wheel_diameter>0.1</wheel_diameter>
+            <wheel_diameter>0.107</wheel_diameter>
             <!-- Limits -->
             <max_wheel_torque>200</max_wheel_torque>

File: src/description/gazebo_control_skid.xacro (robot description, xacro)
@@ -5,5 +5,5 @@
             <ros>
             <namespace>/</namespace>
-            <remapping>cmd_vel:=cmd_vel</remapping>
+            <remapping>cmd_vel:=/diff_cont/cmd_vel_unstamped</remapping>
             <remapping>odom:=odom</remapping>
             </ros>
@@ -19,6 +19,6 @@
             <wheel_separation>0.415</wheel_separation>
             <wheel_separation>0.415</wheel_separation>
-            <wheel_diameter>0.1</wheel_diameter>
-            <wheel_diameter>0.1</wheel_diameter>
+            <wheel_diameter>0.107</wheel_diameter>
+            <wheel_diameter>0.107</wheel_diameter>
             <!-- limits -->
             <max_wheel_torque>200</max_wheel_torque>

File: src/description/robot.urdf.xacro (robot description, xacro)
@@ -4,5 +4,5 @@
         on launch_sim.lauch.py on line 28 -->
     <xacro:arg name="use_ros2_control" default="true"/>
-    <xacro:arg name="sim_mode" default="true"/>
+    <xacro:arg name="sim_mode" default="false"/>
     <xacro:include filename="robot_core.xacro" />
     <xacro:if value="$(arg use_ros2_control)">

File: src/description/robot_core.xacro (robot description, xacro)
@@ -172,5 +172,5 @@
       <origin rpy="-1.57079635 0 0" xyz="0 0 0"/>
       <geometry>
-        <sphere radius="0.111"/> <!-- <cylinder length="0.075" radius="0.111"/> -->
+        <sphere radius="0.107"/> <!-- <cylinder length="0.075" radius="0.111"/> -->
       </geometry>
     </collision>
@@ -241,5 +241,5 @@
       <origin rpy="-1.57079635 0 0" xyz="0 0 0"/>
       <geometry>
-        <sphere radius="0.111"/> <!-- <cylinder length="0.075" radius="0.111"/> -->
+        <sphere radius="0.107"/> <!-- <cylinder length="0.075" radius="0.111"/> -->
       </geometry>
     </collision>
@@ -310,5 +310,5 @@
       <origin rpy="-1.57079635 0 0" xyz="0 0 0"/>
       <geometry>
-        <sphere radius="0.111"/> <!-- <cylinder length="0.075" radius="0.111"/> -->
+        <sphere radius="0.107"/> <!-- <cylinder length="0.075" radius="0.111"/> -->
       </geometry>
     </collision>
@@ -379,5 +379,5 @@
       <origin rpy="-1.57079635 0 0" xyz="0 0 0"/>
       <geometry>
-        <sphere radius="0.111"/> <!-- <cylinder length="0.075" radius="0.111"/> -->
+        <sphere radius="0.107"/> <!-- <cylinder length="0.075" radius="0.111"/> -->
       </geometry>
     </collision>

File: src/description/ros2_control.xacro (robot description, xacro)
@@ -13,5 +13,5 @@
                 <param name="baud_rate">57600</param>
                 <param name="timeout">1000</param>
-                <param name="enc_counts_per_rev">34000</param>
+                <param name="enc_counts_per_rev">35000</param>
                 <!-- encoder= mas o menos =34800 -->
             </hardware>
