Commit message: some compatibility changes

File: src/description/robot_core.xacro (robot description, xacro)
@@ -106,5 +106,5 @@
     <visual>
       <geometry>
-        <mesh filename="$(find higgs2)/src/meshes/sonar_trasero.stl"/>
+        <mesh filename="file://src/meshes/sonar_trasero.stl"/>
       </geometry>
       <origin rpy="0 0 0" xyz="0 0 0"/>
@@ -113,5 +113,5 @@
     <collision>
       <geometry>
-        <mesh filename="$(find higgs2)/src/meshes/sonar_trasero.stl"/>
+        <mesh filename="file://src/meshes/sonar_trasero.stl"/>
       </geometry>
       <origin rpy="0 0 0" xyz="0 0 0"/>
@@ -140,12 +140,12 @@
       <origin rpy="0 0 0" xyz="0 0 0"/>
       <geometry>
-         <mesh filename="$(find higgs2)/src/meshes/eje.stl"/>
-      </geometry>
-      <material name="black"/>
-    </visual>
-    <collision>
-      <origin rpy="0 0 0" xyz="0 0 0"/>
-      <geometry>
-        <mesh filename="$(find higgs2)/src/meshes/eje.stl"/>
+         <mesh filename="file://src/meshes/eje.stl"/>
+      </geometry>
+      <material name="black"/>
+    </visual>
+    <collision>
+      <origin rpy="0 0 0" xyz="0 0 0"/>
+      <geometry>
+        <mesh filename="file://src/meshes/eje.stl"/>
       </geometry>
     </collision>
@@ -165,5 +165,5 @@
       <origin rpy="0 0 0" xyz="0 0 0"/>
       <geometry>
-         <mesh filename="$(find higgs2)/src/meshes/rueda.stl"/>
+         <mesh filename="file://src/meshes/rueda.stl"/>
       </geometry>
       <material name="black"/>
@@ -209,12 +209,12 @@
       <origin rpy="0 0 0" xyz="0 0 0"/>
       <geometry>
-         <mesh filename="$(find higgs2)/src/meshes/eje.stl"/>
-      </geometry>
-      <material name="black"/>
-    </visual>
-    <collision>
-      <origin rpy="0 0 0" xyz="0 0 0"/>
-      <geometry>
-        <mesh filename="$(find higgs2)/src/meshes/eje.stl"/>
+         <mesh filename="file://src/meshes/eje.stl"/>
+      </geometry>
+      <material name="black"/>
+    </visual>
+    <collision>
+      <origin rpy="0 0 0" xyz="0 0 0"/>
+      <geometry>
+        <mesh filename="file://src/meshes/eje.stl"/>
       </geometry>
     </collision>
@@ -234,5 +234,5 @@
       <origin rpy="0 0 0" xyz="0 0 0"/>
       <geometry>
-        <mesh filename="$(find higgs2)/src/meshes/rueda.stl"/>
+        <mesh filename="file://src/meshes/rueda.stl"/>
       </geometry>
       <material name="black"/>
@@ -278,12 +278,12 @@
       <origin rpy="0 0 0" xyz="0 0 0"/>
       <geometry>
-         <mesh filename="$(find higgs2)/src/meshes/eje.stl"/>
-      </geometry>
-      <material name="black"/>
-    </visual>
-    <collision>
-      <origin rpy="0 0 0" xyz="0 0 0"/>
-      <geometry>
-        <mesh filename="$(find higgs2)/src/meshes/eje.stl"/>
+         <mesh filename="file://src/meshes/eje.stl"/>
+      </geometry>
+      <material name="black"/>
+    </visual>
+    <collision>
+      <origin rpy="0 0 0" xyz="0 0 0"/>
+      <geometry>
+        <mesh filename="file://src/meshes/eje.stl"/>
       </geometry>
     </collision>
@@ -303,5 +303,5 @@
       <origin rpy="0 0 0" xyz="0 0 0"/>
       <geometry>
-        <mesh filename="$(find higgs2)/src/meshes/rueda.stl"/>
+        <mesh filename="file://src/meshes/rueda.stl"/>
       </geometry>
       <material name="black"/>
@@ -347,12 +347,12 @@
       <origin rpy="0 0 0" xyz="0 0 0"/>
       <geometry>
-         <mesh filename="$(find higgs2)/src/meshes/eje.stl"/>
-      </geometry>
-      <material name="black"/>
-    </visual>
-    <collision>
-      <origin rpy="0 0 0" xyz="0 0 0"/>
-      <geometry>
-        <mesh filename="$(find higgs2)/src/meshes/eje.stl"/>
+         <mesh filename="file://src/meshes/eje.stl"/>
+      </geometry>
+      <material name="black"/>
+    </visual>
+    <collision>
+      <origin rpy="0 0 0" xyz="0 0 0"/>
+      <geometry>
+        <mesh filename="file://src/meshes/eje.stl"/>
       </geometry>
     </collision>
@@ -372,5 +372,5 @@
       <origin rpy="0 0 0" xyz="0 0 0"/>
       <geometry>
-        <mesh filename="$(find higgs2)/src/meshes/rueda.stl"/>
+        <mesh filename="file://src/meshes/rueda.stl"/>
       </geometry>
       <material name="black"/>

Commit message: joints not working

File: src/description/robot_core.xacro (robot description, xacro)
@@ -130,5 +130,5 @@
 <!-- =================================================================================== -->
 <link name="Eje_izq_delantero_link">
-      <visual>
+    <visual>
       <origin rpy="0 0 0" xyz="0 0 0"/>
       <geometry>
@@ -155,5 +155,5 @@
 </joint>
 <link name="Rueda_izq_delantera_link">
-      <visual>
+    <visual>
       <origin rpy="0 0 0" xyz="0 0 0"/>
       <geometry>
@@ -175,7 +175,7 @@
   </link>
 <joint name="base_ruedaizqdel_joint" type="continuous">
-    <axis xyz="0 1 0"/>
+    <axis rpy="0 0 0" xyz="0 1 0"/>
     <!--<limit effort="80" velocity="0.268"/>-->
-    <joint_properties damping="0.7"/>
+    <!-- <joint_properties damping="0.7"/> -->
     <origin rpy="0 0 0" xyz="0 0.041 0"/>
     <parent link="Eje_izq_delantero_link"/>
@@ -220,5 +220,5 @@
   </joint>
 <link name="Rueda_der_delantera_link">
-      <visual>
+    <visual>
       <origin rpy="0 0 0" xyz="0 0 0"/>
       <geometry>
@@ -344,5 +344,5 @@
     </inertial>
   </link>
-   <joint name="base_eje_der_trasero_joint" type="fixed">
+<joint name="base_eje_der_trasero_joint" type="fixed">
     <origin rpy="0 0 0" xyz="-0.135 -0.156 0.111"/>
     <parent link="base_link"/>
@@ -466,6 +466,6 @@
       <visual>
             <material>
-                <ambient>.3 .3 .3  1.0</ambient>
-                <diffuse>.7 .7 .7  1.0</diffuse>
+                <ambient>0.3 0.3 0.3 1.0</ambient>
+                <diffuse>0.7 0.7 0.7 1.0</diffuse>
                 <specular>0.01 0.01 0.01 1.0 1.5</specular>
             </material>
