Commit message: ros2_control working

File: src/description/lidar.xacro (robot description, xacro)
@@ -59,6 +59,9 @@
       <plugin name="gazebo_ros_head_hokuyo_controller" filename="libgazebo_ros_ray_sensor.so">
         <ros>
+            <!-- <argument>~/out:=scan</argument> -->
+            <argument>--ros-args</argument>
+            <argument>-r</argument>
             <argument>~/out:=scan</argument>
-              </ros>
+        </ros>
         <output_type>sensor_msgs/LaserScan</output_type>
         <topicName>/laser/scan</topicName>

File: src/description/robot.urdf.xacro (robot description, xacro)
@@ -3,5 +3,5 @@
     <!-- To change the control between ros2 or skid, change the next true or false and change
         on launch_sim.lauch.py on line 28 -->
-    <xacro:arg name="use_ros2_control" default="false"/>
+    <xacro:arg name="use_ros2_control" default="true"/>
     <xacro:arg name="sim_mode" default="true"/>
     <xacro:include filename="robot_core.xacro" />

File: src/description/robot_core.xacro (robot description, xacro)
@@ -172,5 +172,5 @@
       <origin rpy="-1.57079635 0 0" xyz="0 0 0"/>
       <geometry>
-        <cylinder length="0.075" radius="0.111"/>
+        <sphere radius="0.111"/> <!-- <cylinder length="0.075" radius="0.111"/> -->
       </geometry>
     </collision>
@@ -190,11 +190,11 @@
   </joint>
 <gazebo reference="Rueda_izq_delantera_link">
-      <mu1 value="200.0"/>
+      <!-- <mu1 value="200.0"/>
       <mu2 value="100.0"/>
       <kp value="10000000.0" />
-      <kd value="1.0" />
+      <kd value="1.0" /> -->
       <material>Gazebo/Grey</material>
     </gazebo>
-<transmission name="rueda_izq_delantera">
+<!-- <transmission name="rueda_izq_delantera">
     <type>transmission_interface/SimpleTransmission</type>
     <actuator name="rueda_izq_del_motor">
@@ -204,5 +204,5 @@
       <hardwareInterface>hardware_interface/VelocityJointInterface</hardwareInterface>
     </joint>
-  </transmission>
+  </transmission> -->
 <link name="Eje_der_delantero_link">
       <visual>
@@ -241,5 +241,5 @@
       <origin rpy="-1.57079635 0 0" xyz="0 0 0"/>
       <geometry>
-        <cylinder length="0.075" radius="0.111"/>
+        <sphere radius="0.111"/> <!-- <cylinder length="0.075" radius="0.111"/> -->
       </geometry>
     </collision>
@@ -259,11 +259,11 @@
   </joint>
 <gazebo reference="Rueda_der_delantera_link">
-      <mu1 value="200.0"/>
+      <!-- <mu1 value="200.0"/>
       <mu2 value="100.0"/>
       <kp value="10000000.0" />
-      <kd value="1.0" />
+      <kd value="1.0" /> -->
       <material>Gazebo/Grey</material>
     </gazebo>
-<transmission name="rueda_der_delantera">
+<!-- <transmission name="rueda_der_delantera">
     <type>transmission_interface/SimpleTransmission</type>
     <actuator name="rueda_der_del_motor">
@@ -273,5 +273,5 @@
       <hardwareInterface>hardware_interface/VelocityJointInterface</hardwareInterface>
     </joint>
-  </transmission>
+  </transmission> -->
 <link name="Eje_izq_trasero_link">
       <visual>
@@ -310,5 +310,5 @@
       <origin rpy="-1.57079635 0 0" xyz="0 0 0"/>
       <geometry>
-        <cylinder length="0.075" radius="0.111"/>
+        <sphere radius="0.111"/> <!-- <cylinder length="0.075" radius="0.111"/> -->
       </geometry>
     </collision>
@@ -328,11 +328,11 @@
   </joint>
 <gazebo reference="Rueda_izq_trasera_link">
-      <mu1 value="200.0"/>   <!--200.0 y 100.0-->
+      <!-- <mu1 value="200.0"/>
       <mu2 value="100.0"/>
       <kp value="10000000.0" />
-      <kd value="1.0" />
+      <kd value="1.0" /> -->
       <material>Gazebo/Grey</material>
     </gazebo>
-<transmission name="rueda_izq_trasera">
+<!-- <transmission name="rueda_izq_trasera">
     <type>transmission_interface/SimpleTransmission</type>
     <actuator name="rueda_izq_tra_motor">
@@ -342,5 +342,5 @@
       <hardwareInterface>hardware_interface/VelocityJointInterface</hardwareInterface>
     </joint>
-  </transmission>
+  </transmission> -->
 <link name="Eje_der_trasero_link">
       <visual>
@@ -379,5 +379,5 @@
       <origin rpy="-1.57079635 0 0" xyz="0 0 0"/>
       <geometry>
-        <cylinder length="0.075" radius="0.111"/>
+        <sphere radius="0.111"/> <!-- <cylinder length="0.075" radius="0.111"/> -->
       </geometry>
     </collision>
@@ -397,11 +397,11 @@
   </joint>
 <gazebo reference="Rueda_der_trasera_link">
-      <mu1 value="200.0"/>   <!--200.0 y 100.0-->
+      <!-- <mu1 value="200.0"/>
       <mu2 value="100.0"/>
       <kp value="10000000.0" />
-      <kd value="1.0" />
+      <kd value="1.0" /> -->
       <material>Gazebo/Grey</material>
     </gazebo>
-<transmission name="rueda_der_trasera">
+<!-- <transmission name="rueda_der_trasera">
     <type>transmission_interface/SimpleTransmission</type>
     <actuator name="rueda_der_tra_motor">
@@ -411,12 +411,5 @@
       <hardwareInterface>hardware_interface/VelocityJointInterface</hardwareInterface>
     </joint>
-  </transmission>
-   <!-- Gazebo plugin for ROS Control -->
-  <gazebo>
-    <plugin name="gazebo_ros_control" filename="libgazebo_ros_control.so">
-      <robotNamespace>/</robotNamespace>
-      <robotSimType>gazebo_ros_control/DefaultRobotHWSim</robotSimType>
-    </plugin>
-  </gazebo>
+  </transmission> -->
 <gazebo reference="base_link">
       <material>Gazebo/Red</material>

Commit message: real robot test

File: src/description/lidar.xacro (robot description, xacro)
@@ -6,5 +6,5 @@
       <origin xyz="0 0 0" rpy="0 0 0"/>
       <geometry>
-    <mesh filename="file://src/meshes/hokuyo.dae"/>
+    <mesh filename="$(find higgs2)/src/meshes/hokuyo.dae"/>
       </geometry>
     </collision>
@@ -12,5 +12,5 @@
       <origin xyz="0 0 0" rpy="0 0 0"/>
       <geometry>
-        <mesh filename="file://src/meshes/hokuyo.dae"/>
+        <mesh filename="$(find higgs2)/src/meshes/hokuyo.dae"/>
       </geometry>
     </visual>

File: src/description/robot_core.xacro (robot description, xacro)
@@ -106,5 +106,5 @@
     <visual>
       <geometry>
-        <mesh filename="file://src/meshes/sonar_trasero.stl"/>
+        <mesh filename="$(find higgs2)/src/meshes/sonar_trasero.stl"/>
       </geometry>
       <origin rpy="0 0 0" xyz="0 0 0"/>
@@ -113,5 +113,5 @@
     <collision>
       <geometry>
-        <mesh filename="file://src/meshes/sonar_trasero.stl"/>
+        <mesh filename="$(find higgs2)/src/meshes/sonar_trasero.stl"/>
       </geometry>
       <origin rpy="0 0 0" xyz="0 0 0"/>
@@ -140,12 +140,12 @@
       <origin rpy="0 0 0" xyz="0 0 0"/>
       <geometry>
-         <mesh filename="file://src/meshes/eje.stl"/>
-      </geometry>
-      <material name="black"/>
-    </visual>
-    <collision>
-      <origin rpy="0 0 0" xyz="0 0 0"/>
-      <geometry>
-        <mesh filename="file://src/meshes/eje.stl"/>
+         <mesh filename="$(find higgs2)/src/meshes/eje.stl"/>
+      </geometry>
+      <material name="black"/>
+    </visual>
+    <collision>
+      <origin rpy="0 0 0" xyz="0 0 0"/>
+      <geometry>
+        <mesh filename="$(find higgs2)/src/meshes/eje.stl"/>
       </geometry>
     </collision>
@@ -165,5 +165,5 @@
       <origin rpy="0 0 0" xyz="0 0 0"/>
       <geometry>
-         <mesh filename="file://src/meshes/rueda.stl"/>
+         <mesh filename="$(find higgs2)/src/meshes/rueda.stl"/>
       </geometry>
       <material name="black"/>
@@ -209,12 +209,12 @@
       <origin rpy="0 0 0" xyz="0 0 0"/>
       <geometry>
-         <mesh filename="file://src/meshes/eje.stl"/>
-      </geometry>
-      <material name="black"/>
-    </visual>
-    <collision>
-      <origin rpy="0 0 0" xyz="0 0 0"/>
-      <geometry>
-        <mesh filename="file://src/meshes/eje.stl"/>
+         <mesh filename="$(find higgs2)/src/meshes/eje.stl"/>
+      </geometry>
+      <material name="black"/>
+    </visual>
+    <collision>
+      <origin rpy="0 0 0" xyz="0 0 0"/>
+      <geometry>
+        <mesh filename="$(find higgs2)/src/meshes/eje.stl"/>
       </geometry>
     </collision>
@@ -234,5 +234,5 @@
       <origin rpy="0 0 0" xyz="0 0 0"/>
       <geometry>
-        <mesh filename="file://src/meshes/rueda.stl"/>
+        <mesh filename="$(find higgs2)/src/meshes/rueda.stl"/>
       </geometry>
       <material name="black"/>
@@ -278,12 +278,12 @@
       <origin rpy="0 0 0" xyz="0 0 0"/>
       <geometry>
-         <mesh filename="file://src/meshes/eje.stl"/>
-      </geometry>
-      <material name="black"/>
-    </visual>
-    <collision>
-      <origin rpy="0 0 0" xyz="0 0 0"/>
-      <geometry>
-        <mesh filename="file://src/meshes/eje.stl"/>
+         <mesh filename="$(find higgs2)/src/meshes/eje.stl"/>
+      </geometry>
+      <material name="black"/>
+    </visual>
+    <collision>
+      <origin rpy="0 0 0" xyz="0 0 0"/>
+      <geometry>
+        <mesh filename="$(find higgs2)/src/meshes/eje.stl"/>
       </geometry>
     </collision>
@@ -303,5 +303,5 @@
       <origin rpy="0 0 0" xyz="0 0 0"/>
       <geometry>
-        <mesh filename="file://src/meshes/rueda.stl"/>
+        <mesh filename="$(find higgs2)/src/meshes/rueda.stl"/>
       </geometry>
       <material name="black"/>
@@ -347,12 +347,12 @@
       <origin rpy="0 0 0" xyz="0 0 0"/>
       <geometry>
-         <mesh filename="file://src/meshes/eje.stl"/>
-      </geometry>
-      <material name="black"/>
-    </visual>
-    <collision>
-      <origin rpy="0 0 0" xyz="0 0 0"/>
-      <geometry>
-        <mesh filename="file://src/meshes/eje.stl"/>
+         <mesh filename="$(find higgs2)/src/meshes/eje.stl"/>
+      </geometry>
+      <material name="black"/>
+    </visual>
+    <collision>
+      <origin rpy="0 0 0" xyz="0 0 0"/>
+      <geometry>
+        <mesh filename="$(find higgs2)/src/meshes/eje.stl"/>
       </geometry>
     </collision>
@@ -372,5 +372,5 @@
       <origin rpy="0 0 0" xyz="0 0 0"/>
       <geometry>
-        <mesh filename="file://src/meshes/rueda.stl"/>
+        <mesh filename="$(find higgs2)/src/meshes/rueda.stl"/>
       </geometry>
       <material name="black"/>

File: src/description/ros2_control.xacro (robot description, xacro)
@@ -13,5 +13,6 @@
                 <param name="baud_rate">57600</param>
                 <param name="timeout">1000</param>
-                <param name="enc_counts_per_rev">3436</param>
+                <param name="enc_counts_per_rev">32500</param>
+                <!-- encoder= mas o menos =34800 -->
             </hardware>
             <joint name="base_ruedaizqdel_joint">

Commit message: nav2 working

File: src/description/lidar.xacro (robot description, xacro)
@@ -6,5 +6,5 @@
       <origin xyz="0 0 0" rpy="0 0 0"/>
       <geometry>
-    <mesh filename="file://src/meshes/hokuyo.dae"/>
+    <mesh filename="$(find higgs2)/src/meshes/hokuyo.dae"/>
       </geometry>
     </collision>
@@ -12,5 +12,5 @@
       <origin xyz="0 0 0" rpy="0 0 0"/>
       <geometry>
-        <mesh filename="file://src/meshes/hokuyo.dae"/>
+        <mesh filename="$(find higgs2)/src/meshes/hokuyo.dae"/>
       </geometry>
     </visual>
@@ -32,5 +32,5 @@
       <pose>0 0 0 0 0 0</pose>
       <visualize>true</visualize>
-      <update_rate>40</update_rate>
+      <update_rate>10</update_rate>
       <ray>
         <scan>
@@ -59,11 +59,11 @@
       <plugin name="gazebo_ros_head_hokuyo_controller" filename="libgazebo_ros_ray_sensor.so">
         <ros>
-            <!-- <argument>~/out:=scan</argument> -->
-            <argument>--ros-args</argument>
+            <argument>~/out:=scan</argument>
+            <!-- <argument>- -ros-args</argument>
             <argument>-r</argument>
-            <argument>~/out:=scan</argument>
+            <argument>~/out:=scan</argument> -->
         </ros>
         <output_type>sensor_msgs/LaserScan</output_type>
-        <topicName>/laser/scan</topicName>
+        <!-- <topicName>/laser/scan</topicName> -->
         <frameName>hokuyo_link</frameName>
         <visualize>true</visualize>

File: src/description/ros2_control.xacro (robot description, xacro)
@@ -91,4 +91,5 @@
         <plugin name="gazebo_ros2_control" filename="libgazebo_ros2_control.so">
             <parameters>$(find higgs2)/config/my_controllers.yaml</parameters>
+            <parameters>$(find higgs2)/config/gaz_ros2_ctl_use_sim.yaml</parameters>
         </plugin>
     </gazebo>

Commit message: joystick test and rviz2 correct

File: src/description/lidar.xacro (robot description, xacro)
@@ -6,5 +6,5 @@
       <origin xyz="0 0 0" rpy="0 0 0"/>
       <geometry>
-    <mesh filename="$(find higgs2)/src/meshes/hokuyo.dae"/>
+    <mesh filename="file://$(find higgs2)/src/meshes/hokuyo.dae"/>
       </geometry>
     </collision>
@@ -12,5 +12,5 @@
       <origin xyz="0 0 0" rpy="0 0 0"/>
       <geometry>
-        <mesh filename="$(find higgs2)/src/meshes/hokuyo.dae"/>
+        <mesh filename="file://$(find higgs2)/src/meshes/hokuyo.dae"/>
       </geometry>
     </visual>

File: src/description/robot_core.xacro (robot description, xacro)
@@ -34,5 +34,5 @@
     <visual>
       <geometry>
-        <mesh filename="$(find higgs2)/src/meshes/chasis.dae"/>
+        <mesh filename="file://$(find higgs2)/src/meshes/chasis.dae"/>
       </geometry>
       <origin rpy="0 0 0" xyz="0 0 0.177"/>
@@ -57,5 +57,5 @@
     <visual>
       <geometry>
-        <mesh filename="$(find higgs2)/src/meshes/cubierta.dae"/>
+        <mesh filename="file://$(find higgs2)/src/meshes/cubierta.dae"/>
         <origin rpy="0 0 0" xyz="0 0 0"/>
       </geometry>
@@ -84,5 +84,5 @@
     <visual>
       <geometry>
-        <mesh filename="$(find higgs2)/src/meshes/sonar_delantero.dae"/>
+        <mesh filename="file://$(find higgs2)/src/meshes/sonar_delantero.dae"/>
       </geometry>
       <origin rpy="0 0 0" xyz="0 0 0"/>
@@ -91,5 +91,5 @@
     <collision>
       <geometry>
-        <mesh filename="$(find higgs2)/src/meshes/sonar_delantero.dae"/>
+        <mesh filename="file://$(find higgs2)/src/meshes/sonar_delantero.dae"/>
       </geometry>
       <origin rpy="0 0 0" xyz="0 0 0"/>
@@ -106,5 +106,5 @@
     <visual>
       <geometry>
-        <mesh filename="$(find higgs2)/src/meshes/sonar_trasero.stl"/>
+        <mesh filename="file://$(find higgs2)/src/meshes/sonar_trasero.stl"/>
       </geometry>
       <origin rpy="0 0 0" xyz="0 0 0"/>
@@ -113,5 +113,5 @@
     <collision>
       <geometry>
-        <mesh filename="$(find higgs2)/src/meshes/sonar_trasero.stl"/>
+        <mesh filename="file://$(find higgs2)/src/meshes/sonar_trasero.stl"/>
       </geometry>
       <origin rpy="0 0 0" xyz="0 0 0"/>
@@ -140,12 +140,12 @@
       <origin rpy="0 0 0" xyz="0 0 0"/>
       <geometry>
-         <mesh filename="$(find higgs2)/src/meshes/eje.stl"/>
-      </geometry>
-      <material name="black"/>
-    </visual>
-    <collision>
-      <origin rpy="0 0 0" xyz="0 0 0"/>
-      <geometry>
-        <mesh filename="$(find higgs2)/src/meshes/eje.stl"/>
+         <mesh filename="file://$(find higgs2)/src/meshes/eje.stl"/>
+      </geometry>
+      <material name="black"/>
+    </visual>
+    <collision>
+      <origin rpy="0 0 0" xyz="0 0 0"/>
+      <geometry>
+        <mesh filename="file://$(find higgs2)/src/meshes/eje.stl"/>
       </geometry>
     </collision>
@@ -165,5 +165,5 @@
       <origin rpy="0 0 0" xyz="0 0 0"/>
       <geometry>
-         <mesh filename="$(find higgs2)/src/meshes/rueda.stl"/>
+         <mesh filename="file://$(find higgs2)/src/meshes/rueda.stl"/>
       </geometry>
       <material name="black"/>
@@ -209,12 +209,12 @@
       <origin rpy="0 0 0" xyz="0 0 0"/>
       <geometry>
-         <mesh filename="$(find higgs2)/src/meshes/eje.stl"/>
-      </geometry>
-      <material name="black"/>
-    </visual>
-    <collision>
-      <origin rpy="0 0 0" xyz="0 0 0"/>
-      <geometry>
-        <mesh filename="$(find higgs2)/src/meshes/eje.stl"/>
+         <mesh filename="file://$(find higgs2)/src/meshes/eje.stl"/>
+      </geometry>
+      <material name="black"/>
+    </visual>
+    <collision>
+      <origin rpy="0 0 0" xyz="0 0 0"/>
+      <geometry>
+        <mesh filename="file://$(find higgs2)/src/meshes/eje.stl"/>
       </geometry>
     </collision>
@@ -234,5 +234,5 @@
       <origin rpy="0 0 0" xyz="0 0 0"/>
       <geometry>
-        <mesh filename="$(find higgs2)/src/meshes/rueda.stl"/>
+        <mesh filename="file://$(find higgs2)/src/meshes/rueda.stl"/>
       </geometry>
       <material name="black"/>
@@ -278,12 +278,12 @@
       <origin rpy="0 0 0" xyz="0 0 0"/>
       <geometry>
-         <mesh filename="$(find higgs2)/src/meshes/eje.stl"/>
-      </geometry>
-      <material name="black"/>
-    </visual>
-    <collision>
-      <origin rpy="0 0 0" xyz="0 0 0"/>
-      <geometry>
-        <mesh filename="$(find higgs2)/src/meshes/eje.stl"/>
+         <mesh filename="file://$(find higgs2)/src/meshes/eje.stl"/>
+      </geometry>
+      <material name="black"/>
+    </visual>
+    <collision>
+      <origin rpy="0 0 0" xyz="0 0 0"/>
+      <geometry>
+        <mesh filename="file://$(find higgs2)/src/meshes/eje.stl"/>
       </geometry>
     </collision>
@@ -303,5 +303,5 @@
       <origin rpy="0 0 0" xyz="0 0 0"/>
       <geometry>
-        <mesh filename="$(find higgs2)/src/meshes/rueda.stl"/>
+        <mesh filename="file://$(find higgs2)/src/meshes/rueda.stl"/>
       </geometry>
       <material name="black"/>
@@ -347,12 +347,12 @@
       <origin rpy="0 0 0" xyz="0 0 0"/>
       <geometry>
-         <mesh filename="$(find higgs2)/src/meshes/eje.stl"/>
-      </geometry>
-      <material name="black"/>
-    </visual>
-    <collision>
-      <origin rpy="0 0 0" xyz="0 0 0"/>
-      <geometry>
-        <mesh filename="$(find higgs2)/src/meshes/eje.stl"/>
+         <mesh filename="file://$(find higgs2)/src/meshes/eje.stl"/>
+      </geometry>
+      <material name="black"/>
+    </visual>
+    <collision>
+      <origin rpy="0 0 0" xyz="0 0 0"/>
+      <geometry>
+        <mesh filename="file://$(find higgs2)/src/meshes/eje.stl"/>
       </geometry>
     </collision>
@@ -372,5 +372,5 @@
       <origin rpy="0 0 0" xyz="0 0 0"/>
       <geometry>
-        <mesh filename="$(find higgs2)/src/meshes/rueda.stl"/>
+        <mesh filename="file://$(find higgs2)/src/meshes/rueda.stl"/>
       </geometry>
       <material name="black"/>

File: src/description/ros2_control.xacro (robot description, xacro)
@@ -13,5 +13,5 @@
                 <param name="baud_rate">57600</param>
                 <param name="timeout">1000</param>
-                <param name="enc_counts_per_rev">3436</param>
+                <param name="enc_counts_per_rev">34000</param>
             </hardware>
             <joint name="base_ruedaizqdel_joint">
