Commit message: first draft

File: src/description/lidar.xacro (robot description, xacro)
@@ -1,4 +1,4 @@
 <?xml version="1.0"?>
-<robot xmlns:xacro="http://www.ros.org/wiki/xacro" name="Pioneer_2-AT_8">
+<robot xmlns:xacro="http://www.ros.org/wiki/xacro">
 <!--Lidar sensor: -->
 <link name="hokuyo_link">
@@ -6,5 +6,5 @@
       <origin xyz="0 0 0" rpy="0 0 0"/>
       <geometry>
-    <mesh filename="file://$(find higgs2)/src/meshes/hokuyo.dae"/>
+        <mesh filename="file://$(find higgs2)/src/meshes/hokuyo.dae"/>
       </geometry>
     </collision>
@@ -30,5 +30,8 @@
 <gazebo reference="hokuyo_link">
     <sensor type="ray" name="head_hokuyo_sensor">
-      <pose>0 0 0 0 0 0</pose>
+      <!-- <pose>0 0 0 0 0 0</pose> -->
+      <topic>/laserscan</topic>
+      <always_on>true</always_on>
+      <always_on>1</always_on>
       <visualize>true</visualize>
       <update_rate>10</update_rate>
@@ -57,17 +60,4 @@
         </noise>
       </ray>
-      <plugin name="gazebo_ros_head_hokuyo_controller" filename="libgazebo_ros_ray_sensor.so">
-        <ros>
-            <!-- <argument>~/out:=scan</argument> -->
-            <argument>--ros-args</argument>
-            <argument>-r</argument>
-            <argument>~/out:=scan</argument>
-        </ros>
-        <output_type>sensor_msgs/LaserScan</output_type>
-        <!-- <topicName>/laser/scan</topicName> -->
-        <frameName>hokuyo_link</frameName>
-        <visualize>true</visualize>
-        <always_on>1</always_on>
-      </plugin>
     </sensor>
   </gazebo>

File: src/description/robot.urdf.xacro (robot description, xacro)
@@ -1,15 +1,17 @@
 <?xml version="1.0"?>
-<robot xmlns:xacro="http://www.ros.org/wiki/xacro"  name="Pioneer_2-AT_8" >
+<robot xmlns:xacro="http://www.ros.org/wiki/xacro"  name="higgs2_sim" >
     <!-- To change the control between ros2 or skid, change the next true or false and change
         on launch_sim.lauch.py on line 28 -->
-    <xacro:arg name="use_ros2_control" default="true"/>
-    <xacro:arg name="sim_mode" default="true"/>
-    <xacro:include filename="robot_core.xacro" />
-    <xacro:if value="$(arg use_ros2_control)">
+    <!-- <xacro:arg name="use_ros2_control" default="false"/>
+    <xacro:arg name="sim_mode" default="true"/> -->
+    <!-- <xacro:if value="$(arg use_ros2_control)">
         <xacro:include filename="ros2_control.xacro" />
     </xacro:if>
     <xacro:unless value="$(arg use_ros2_control)">
         <xacro:include filename="gazebo_control_skid.xacro" />
-    </xacro:unless>
-    <xacro:include filename="lidar.xacro" />
+    </xacro:unless> -->
+    <xacro:include filename="$(find higgs2)/src/description/robot_core.xacro" />
+    <xacro:include filename="$(find higgs2)/src/description/robot.gazebo" />
+    <xacro:include filename="$(find higgs2)/src/description/lidar.xacro" />
+    <xacro:include filename="$(find higgs2)/src/description/materials.xacro" />
 </robot>

File: src/description/robot_core.xacro (robot description, xacro)
@@ -1,17 +1,4 @@
 <?xml version="1.0"?>
 <robot xmlns:xacro="http://www.ros.org/wiki/xacro">
-<!--Se define el color de los materiales utilizados.-->
-  <material name="red">
-    <color rgba="0.851 0.0 0.0 1.0"/>
-  </material>
-  <material name="black">
-    <color rgba="0.038 0.038 0.038 1.0"/>
-  </material>
-  <material name="yellow">
-    <color rgba="0.715 0.583 0.210 1.0"/>
-  </material>
-    <material name="white">
-    <color rgba="1.0 1.0 1.0 1.0"/>
-  </material>
 <!-- Chasis -->
 <link name="base_link0">
@@ -91,5 +78,6 @@
     <collision>
       <geometry>
-        <mesh filename="file://$(find higgs2)/src/meshes/sonar_delantero.dae"/>
+        <!-- <mesh filename="file://$(find higgs2)/src/meshes/sonar_delantero.dae"/> -->
+        <sphere radius="0.01"/> <!-- <cylinder length="0.075" radius="0.111"/> -->
       </geometry>
       <origin rpy="0 0 0" xyz="0 0 0"/>
@@ -135,10 +123,15 @@
     <child link="Sonar_trasero_link"/>
   </joint>
-<!--Ruedas y ejes-->
+<!-- =================================================================================== -->
+<!-- |                                          WHEELS AND JOINTS                      | -->
+<!-- =================================================================================== -->
+<!-- =================================================================================== -->
+<!-- |                                          RUEDA IZQ DEL                          | -->
+<!-- =================================================================================== -->
 <link name="Eje_izq_delantero_link">
       <visual>
       <origin rpy="0 0 0" xyz="0 0 0"/>
       <geometry>
-         <mesh filename="file://$(find higgs2)/src/meshes/eje.stl"/>
+        <mesh filename="file://$(find higgs2)/src/meshes/eje.stl"/>
       </geometry>
       <material name="black"/>
@@ -165,5 +158,5 @@
       <origin rpy="0 0 0" xyz="0 0 0"/>
       <geometry>
-         <mesh filename="file://$(find higgs2)/src/meshes/rueda.stl"/>
+        <mesh filename="file://$(find higgs2)/src/meshes/rueda.stl"/>
       </geometry>
       <material name="black"/>
@@ -189,11 +182,4 @@
     <child link="Rueda_izq_delantera_link"/>
   </joint>
-<gazebo reference="Rueda_izq_delantera_link">
-      <!-- <mu1 value="200.0"/>
-      <mu2 value="100.0"/>
-      <kp value="10000000.0" />
-      <kd value="1.0" /> -->
-      <material>Gazebo/Grey</material>
-    </gazebo>
 <!-- <transmission name="rueda_izq_delantera">
     <type>transmission_interface/SimpleTransmission</type>
@@ -205,9 +191,12 @@
     </joint>
   </transmission> -->
+<!-- =================================================================================== -->
+<!-- |                                          RUEDA DER DEL                          | -->
+<!-- =================================================================================== -->
 <link name="Eje_der_delantero_link">
       <visual>
       <origin rpy="0 0 0" xyz="0 0 0"/>
       <geometry>
-         <mesh filename="file://$(find higgs2)/src/meshes/eje.stl"/>
+        <mesh filename="file://$(find higgs2)/src/meshes/eje.stl"/>
       </geometry>
       <material name="black"/>
@@ -258,11 +247,4 @@
     <child link="Rueda_der_delantera_link"/>
   </joint>
-<gazebo reference="Rueda_der_delantera_link">
-      <!-- <mu1 value="200.0"/>
-      <mu2 value="100.0"/>
-      <kp value="10000000.0" />
-      <kd value="1.0" /> -->
-      <material>Gazebo/Grey</material>
-    </gazebo>
 <!-- <transmission name="rueda_der_delantera">
     <type>transmission_interface/SimpleTransmission</type>
@@ -274,9 +256,12 @@
     </joint>
   </transmission> -->
+<!-- =================================================================================== -->
+<!-- |                                          RUEDA IZQ TRA                          | -->
+<!-- =================================================================================== -->
 <link name="Eje_izq_trasero_link">
       <visual>
       <origin rpy="0 0 0" xyz="0 0 0"/>
       <geometry>
-         <mesh filename="file://$(find higgs2)/src/meshes/eje.stl"/>
+        <mesh filename="file://$(find higgs2)/src/meshes/eje.stl"/>
       </geometry>
       <material name="black"/>
@@ -327,11 +312,4 @@
     <child link="Rueda_izq_trasera_link"/>
   </joint>
-<gazebo reference="Rueda_izq_trasera_link">
-      <!-- <mu1 value="200.0"/>
-      <mu2 value="100.0"/>
-      <kp value="10000000.0" />
-      <kd value="1.0" /> -->
-      <material>Gazebo/Grey</material>
-    </gazebo>
 <!-- <transmission name="rueda_izq_trasera">
     <type>transmission_interface/SimpleTransmission</type>
@@ -343,9 +321,12 @@
     </joint>
   </transmission> -->
+<!-- =================================================================================== -->
+<!-- |                                          RUEDA DER TRA                          | -->
+<!-- =================================================================================== -->
 <link name="Eje_der_trasero_link">
       <visual>
       <origin rpy="0 0 0" xyz="0 0 0"/>
       <geometry>
-         <mesh filename="file://$(find higgs2)/src/meshes/eje.stl"/>
+        <mesh filename="file://$(find higgs2)/src/meshes/eje.stl"/>
       </geometry>
       <material name="black"/>
@@ -396,11 +377,4 @@
     <child link="Rueda_der_trasera_link"/>
   </joint>
-<gazebo reference="Rueda_der_trasera_link">
-      <!-- <mu1 value="200.0"/>
-      <mu2 value="100.0"/>
-      <kp value="10000000.0" />
-      <kd value="1.0" /> -->
-      <material>Gazebo/Grey</material>
-    </gazebo>
 <!-- <transmission name="rueda_der_trasera">
     <type>transmission_interface/SimpleTransmission</type>
@@ -412,27 +386,123 @@
     </joint>
   </transmission> -->
+<!-- =================================================================================== -->
+<!-- |                                          GAZEBO                                 | -->
+<!-- =================================================================================== -->
 <gazebo reference="base_link">
-      <material>Gazebo/Red</material>
+      <!-- <material>Gazebo/Red</material> -->
+      <visual>
+            <material>
+                <ambient>1 0 0 1</ambient>
+                <diffuse>1 0 0 1</diffuse>
+                <specular>0.1 0.1 0.1 1</specular>
+            </material>
+      </visual>
 </gazebo>
 <gazebo reference="cubierta_link">
-      <material>Gazebo/Black</material>
+      <!-- <material>Gazebo/Grey</material> -->
+      <visual>
+            <material>
+                <ambient>.3 .3 .3  1.0</ambient>
+                <diffuse>.7 .7 .7  1.0</diffuse>
+                <specular>0.01 0.01 0.01 1.0 1.5</specular>
+            </material>
+        </visual>
 </gazebo>
 <gazebo reference="Sonar_delantero_link">
-      <material>Gazebo/Yellow</material>
+      <!-- <material>Gazebo/yellow</material> -->
 </gazebo>
 <gazebo reference="Sonar_trasero_link">
-      <material>Gazebo/Yellow</material>
+      <!-- <material>Gazebo/yellow</material> -->
+      <visual>
+            <material>
+                <ambient>0 0 0 1</ambient>
+                <diffuse>0 0 0 1</diffuse>
+                <specular>0.1 0.1 0.1 1 5.0</specular>
+            </material>
+        </visual>
 </gazebo>
 <gazebo reference="Eje_izq_delantero_link">
-      <material>Gazebo/Black</material>
+      <!-- <material>Gazebo/black</material> -->
+      <visual>
+            <material>
+                <ambient>0 0 0 1</ambient>
+                <diffuse>0 0 0 1</diffuse>
+                <specular>0.1 0.1 0.1 1 5.0</specular>
+            </material>
+        </visual>
 </gazebo>
 <gazebo reference="Eje_der_delantero_link">
-      <material>Gazebo/Black</material>
+      <!-- <material>Gazebo/black</material> -->
+      <visual>
+            <material>
+                <ambient>0 0 0 1</ambient>
+                <diffuse>0 0 0 1</diffuse>
+                <specular>0.1 0.1 0.1 1 5.0</specular>
+            </material>
+        </visual>
 </gazebo>
 <gazebo reference="Eje_izq_trasero_link">
-      <material>Gazebo/Black</material>
+      <!-- <material>Gazebo/black</material> -->
+      <visual>
+            <material>
+                <ambient>0 0 0 1</ambient>
+                <diffuse>0 0 0 1</diffuse>
+                <specular>0.1 0.1 0.1 1 5.0</specular>
+            </material>
+        </visual>
 </gazebo>
 <gazebo reference="Eje_der_trasero_link">
-      <material>Gazebo/Black</material>
+      <!-- <material>Gazebo/black</material> -->
+      <visual>
+            <material>
+                <ambient>0 0 0 1</ambient>
+                <diffuse>0 0 0 1</diffuse>
+                <specular>0.1 0.1 0.1 1 5.0</specular>
+            </material>
+        </visual>
+</gazebo>
+<gazebo reference="Rueda_izq_delantera_link">
+      <!-- <material>Gazebo/grey</material> -->
+      <visual>
+            <material>
+                <ambient>.3 .3 .3  1.0</ambient>
+                <diffuse>.7 .7 .7  1.0</diffuse>
+                <specular>0.01 0.01 0.01 1.0 1.5</specular>
+            </material>
+        </visual>
+</gazebo>
+<gazebo reference="Rueda_der_delantera_link">
+      <!-- <material>Gazebo/grey</material> -->
+      <visual>
+            <material>
+                <ambient>.3 .3 .3  1.0</ambient>
+                <diffuse>.7 .7 .7  1.0</diffuse>
+                <specular>0.01 0.01 0.01 1.0 1.5</specular>
+            </material>
+        </visual>
+</gazebo>
+<gazebo reference="Rueda_izq_trasera_link">
+      <!-- <material>Gazebo/grey</material> -->
+      <visual>
+            <material>
+                <ambient>.3 .3 .3  1.0</ambient>
+                <diffuse>.7 .7 .7  1.0</diffuse>
+                <specular>0.01 0.01 0.01 1.0 1.5</specular>
+            </material>
+        </visual>
+</gazebo>
+<gazebo reference="Rueda_der_trasera_link">
+      <!-- <mu1 value="200.0"/>
+      <mu2 value="100.0"/>
+      <kp value="10000000.0" />
+      <kd value="1.0" /> -->
+      <!-- <material>Gazebo/grey</material> -->
+      <visual>
+            <material>
+                <ambient>.3 .3 .3  1.0</ambient>
+                <diffuse>.7 .7 .7  1.0</diffuse>
+                <specular>0.01 0.01 0.01 1.0 1.5</specular>
+            </material>
+        </visual>
 </gazebo>
 </robot>

Commit message: joints working

File: src/description/lidar.xacro (robot description, xacro)
@@ -29,15 +29,15 @@
   <!--Lidar plugin-->
 <gazebo reference="hokuyo_link">
-    <sensor type="ray" name="head_hokuyo_sensor">
+    <sensor type="gpu_lidar" name="head_hokuyo_sensor">
       <!-- <pose>0 0 0 0 0 0</pose> -->
       <topic>/laserscan</topic>
       <always_on>true</always_on>
       <always_on>1</always_on>
-      <visualize>true</visualize>
+      <visualize>false</visualize>
       <update_rate>10</update_rate>
       <ray>
         <scan>
           <horizontal>
-            <samples>360</samples>
+            <samples>720</samples>
             <resolution>1</resolution>
             <min_angle>-3.14</min_angle>
@@ -46,6 +46,6 @@
         </scan>
         <range>
-          <min>1</min>
-          <max>15.0</max>
+          <min>0.5</min>
+          <max>20</max>
           <resolution>0.01</resolution>
         </range>

File: src/description/robot_core.xacro (robot description, xacro)
@@ -1,10 +1,20 @@
 <?xml version="1.0"?>
 <robot xmlns:xacro="http://www.ros.org/wiki/xacro">
-<!-- Chasis -->
-<link name="base_link0">
- </link>
-<!-- Base footprint -->
+<!-- =================================================================================== -->
+<!-- |                                          DUMY LINK                              | -->
+<!-- =================================================================================== -->
+<!-- <link name="base_link0">
+ </link> -->
+ <!-- Parent with no inertia -->
+ <!-- <joint name="chassis_joint" type="fixed">
+        <parent link="base_link0"/>
+        <child link="base_link"/>
+        <origin xyz="-0.1 0 0"/>
+    </joint> -->
+<!-- =================================================================================== -->
+<!-- |                                          BASE FOOTPRINT                         | -->
+<!-- =================================================================================== -->
 <joint name="base_footprint_joint" type="fixed">
-        <parent link="base_link0"/>
+        <parent link="base_link"/>
         <child link="base_footprint"/>
         <origin xyz="0 0 0" rpy="0 0 0"/>
@@ -12,14 +22,11 @@
 <link name="base_footprint">
 </link>
-<!-- Parent with no inertia -->
- <joint name="chassis_joint" type="fixed">
-        <parent link="base_link0"/>
-        <child link="base_link"/>
-        <origin xyz="-0.1 0 0"/>
-    </joint>
+<!-- =================================================================================== -->
+<!-- |                                          CHASIS                                 | -->
+<!-- =================================================================================== -->
 <link name="base_link">
     <visual>
       <geometry>
-        <mesh filename="file://$(find higgs2)/src/meshes/chasis.dae"/>
+        <mesh filename="file://$(find higgs2)/src/meshes/chasis.stl"/>
       </geometry>
       <origin rpy="0 0 0" xyz="0 0 0.177"/>
@@ -40,9 +47,11 @@
     </inertial>
  </link>
-<!-- Cubierta superior -->
+<!-- =================================================================================== -->
+<!-- |                                          CUBIERTA SUPERIOR                      | -->
+<!-- =================================================================================== -->
 <link name="cubierta_link">
     <visual>
       <geometry>
-        <mesh filename="file://$(find higgs2)/src/meshes/cubierta.dae"/>
+        <mesh filename="file://$(find higgs2)/src/meshes/cubierta.stl"/>
         <origin rpy="0 0 0" xyz="0 0 0"/>
       </geometry>
@@ -67,9 +76,11 @@
     <child link="cubierta_link"/>
   </joint>
-<!--Sonar sensor: -->
+<!-- =================================================================================== -->
+<!-- |                                          SONAR SENSORS                          | -->
+<!-- =================================================================================== -->
 <link name="Sonar_delantero_link">
     <visual>
       <geometry>
-        <mesh filename="file://$(find higgs2)/src/meshes/sonar_delantero.dae"/>
+        <mesh filename="file://$(find higgs2)/src/meshes/sonar_delantero.stl"/>
       </geometry>
       <origin rpy="0 0 0" xyz="0 0 0"/>
@@ -78,5 +89,5 @@
     <collision>
       <geometry>
-        <!-- <mesh filename="file://$(find higgs2)/src/meshes/sonar_delantero.dae"/> -->
+        <mesh filename="file://$(find higgs2)/src/meshes/sonar_delantero.stl"/>
         <sphere radius="0.01"/> <!-- <cylinder length="0.075" radius="0.111"/> -->
       </geometry>
@@ -400,18 +411,35 @@
 </gazebo>
 <gazebo reference="cubierta_link">
-      <!-- <material>Gazebo/Grey</material> -->
-      <visual>
-            <material>
-                <ambient>.3 .3 .3  1.0</ambient>
-                <diffuse>.7 .7 .7  1.0</diffuse>
-                <specular>0.01 0.01 0.01 1.0 1.5</specular>
+      <!-- <material>Gazebo/FlatBlack</material> -->
+        <visual>
+            <material>
+                <ambient>0.1 0.1 0.1</ambient>
+                <diffuse>0.1 0.1 0.1</diffuse>
+                <specular>0.01 0.01 0.01 1.0 1.0</specular>
             </material>
         </visual>
 </gazebo>
 <gazebo reference="Sonar_delantero_link">
-      <!-- <material>Gazebo/yellow</material> -->
+      <!-- <material>Gazebo/DarkYellow</material> -->
+      <visual>
+            <material>
+                <ambient>0.7 0.7 0 1</ambient>
+                <diffuse>0.7 0.7 0 1</diffuse>
+                <specular>0 0 0 0 0</specular>
+            </material>
+        </visual>
 </gazebo>
 <gazebo reference="Sonar_trasero_link">
-      <!-- <material>Gazebo/yellow</material> -->
+      <!-- <material>Gazebo/DarkYellow</material> -->
+      <visual>
+            <material>
+                <ambient>0.7 0.7 0 1</ambient>
+                <diffuse>0.7 0.7 0 1</diffuse>
+                <specular>0 0 0 0 0</specular>
+            </material>
+        </visual>
+</gazebo>
+<gazebo reference="Eje_izq_delantero_link">
+      <!-- <material>Gazebo/black</material> -->
       <visual>
             <material>
@@ -422,5 +450,5 @@
         </visual>
 </gazebo>
-<gazebo reference="Eje_izq_delantero_link">
+<gazebo reference="Eje_der_delantero_link">
       <!-- <material>Gazebo/black</material> -->
       <visual>
@@ -432,5 +460,5 @@
         </visual>
 </gazebo>
-<gazebo reference="Eje_der_delantero_link">
+<gazebo reference="Eje_izq_trasero_link">
       <!-- <material>Gazebo/black</material> -->
       <visual>
@@ -442,5 +470,5 @@
         </visual>
 </gazebo>
-<gazebo reference="Eje_izq_trasero_link">
+<gazebo reference="Eje_der_trasero_link">
       <!-- <material>Gazebo/black</material> -->
       <visual>
@@ -452,41 +480,31 @@
         </visual>
 </gazebo>
-<gazebo reference="Eje_der_trasero_link">
-      <!-- <material>Gazebo/black</material> -->
-      <visual>
-            <material>
-                <ambient>0 0 0 1</ambient>
-                <diffuse>0 0 0 1</diffuse>
-                <specular>0.1 0.1 0.1 1 5.0</specular>
-            </material>
-        </visual>
-</gazebo>
 <gazebo reference="Rueda_izq_delantera_link">
-      <!-- <material>Gazebo/grey</material> -->
-      <visual>
-            <material>
-                <ambient>0.3 0.3 0.3 1.0</ambient>
-                <diffuse>0.7 0.7 0.7 1.0</diffuse>
-                <specular>0.01 0.01 0.01 1.0 1.5</specular>
+      <!-- <material>Gazebo/FlatBlack</material> -->
+        <visual>
+            <material>
+                <ambient>0.1 0.1 0.1</ambient>
+                <diffuse>0.1 0.1 0.1</diffuse>
+                <specular>0.01 0.01 0.01 1.0 1.0</specular>
             </material>
         </visual>
 </gazebo>
 <gazebo reference="Rueda_der_delantera_link">
-      <!-- <material>Gazebo/grey</material> -->
-      <visual>
-            <material>
-                <ambient>.3 .3 .3  1.0</ambient>
-                <diffuse>.7 .7 .7  1.0</diffuse>
-                <specular>0.01 0.01 0.01 1.0 1.5</specular>
+      <!-- <material>Gazebo/FlatBlack</material> -->
+        <visual>
+            <material>
+                <ambient>0.1 0.1 0.1</ambient>
+                <diffuse>0.1 0.1 0.1</diffuse>
+                <specular>0.01 0.01 0.01 1.0 1.0</specular>
             </material>
         </visual>
 </gazebo>
 <gazebo reference="Rueda_izq_trasera_link">
-      <!-- <material>Gazebo/grey</material> -->
-      <visual>
-            <material>
-                <ambient>.3 .3 .3  1.0</ambient>
-                <diffuse>.7 .7 .7  1.0</diffuse>
-                <specular>0.01 0.01 0.01 1.0 1.5</specular>
+      <!-- <material>Gazebo/FlatBlack</material> -->
+        <visual>
+            <material>
+                <ambient>0.1 0.1 0.1</ambient>
+                <diffuse>0.1 0.1 0.1</diffuse>
+                <specular>0.01 0.01 0.01 1.0 1.0</specular>
             </material>
         </visual>
@@ -497,10 +515,10 @@
       <kp value="10000000.0" />
       <kd value="1.0" /> -->
-      <!-- <material>Gazebo/grey</material> -->
-      <visual>
-            <material>
-                <ambient>.3 .3 .3  1.0</ambient>
-                <diffuse>.7 .7 .7  1.0</diffuse>
-                <specular>0.01 0.01 0.01 1.0 1.5</specular>
+      <!-- <material>Gazebo/FlatBlack</material> -->
+        <visual>
+            <material>
+                <ambient>0.1 0.1 0.1</ambient>
+                <diffuse>0.1 0.1 0.1</diffuse>
+                <specular>0.01 0.01 0.01 1.0 1.0</specular>
             </material>
         </visual>
