Commit message: nav2 and ball working in sim

File: src/description/lidar.xacro (robot description, xacro)
@@ -23,5 +23,5 @@
  <joint name="hokuyo_joint" type="fixed">
     <axis xyz="0 1 0" />
-    <origin xyz="0.136 0 0.309" rpy="0 0 0"/>
+    <origin xyz="0.05 0 0.309" rpy="0 0 0"/> <!--0.136 x-->
     <parent link="base_link"/>
     <child link="hokuyo_link"/>
