Commit message: change src folder to model

File: model/description/lidar.xacro (robot description, xacro)
@@ -6,5 +6,5 @@
       <origin xyz="0 0 0" rpy="0 0 0"/>
       <geometry>
-        <mesh filename="file://$(find higgs2)/src/meshes/hokuyo.dae"/>
+        <mesh filename="file://$(find higgs2)/model/meshes/hokuyo.dae"/>
       </geometry>
     </collision>
@@ -12,5 +12,5 @@
       <origin xyz="0 0 0" rpy="0 0 0"/>
       <geometry>
-        <mesh filename="file://$(find higgs2)/src/meshes/hokuyo.dae"/>
+        <mesh filename="file://$(find higgs2)/model/meshes/hokuyo.dae"/>
       </geometry>
     </visual>

File: model/description/robot.urdf.xacro (robot description, xacro)
@@ -11,8 +11,8 @@
         <xacro:include filename="gazebo_control_skid.xacro" />
     </xacro:unless> -->
-    <xacro:include filename="$(find higgs2)/src/description/robot_core.xacro" />
-    <xacro:include filename="$(find higgs2)/src/description/robot.gazebo" />
-    <xacro:include filename="$(find higgs2)/src/description/lidar.xacro" />
-    <xacro:include filename="$(find higgs2)/src/description/camera.xacro" />
-    <xacro:include filename="$(find higgs2)/src/description/materials.xacro" />
+    <xacro:include filename="$(find higgs2)/model/description/robot_core.xacro" />
+    <xacro:include filename="$(find higgs2)/model/description/robot.gazebo" />
+    <xacro:include filename="$(find higgs2)/model/description/lidar.xacro" />
+    <xacro:include filename="$(find higgs2)/model/description/camera.xacro" />
+    <xacro:include filename="$(find higgs2)/model/description/materials.xacro" />
 </robot>

File: model/description/robot_core.xacro (robot description, xacro)
@@ -28,5 +28,5 @@
     <visual>
       <geometry>
-        <mesh filename="file://$(find higgs2)/src/meshes/chasis.stl"/>
+        <mesh filename="file://$(find higgs2)/model/meshes/chasis.stl"/>
       </geometry>
       <origin rpy="0 0 0" xyz="0 0 0.177"/>
@@ -53,5 +53,5 @@
     <visual>
       <geometry>
-        <mesh filename="file://$(find higgs2)/src/meshes/cubierta.stl"/>
+        <mesh filename="file://$(find higgs2)/model/meshes/cubierta.stl"/>
         <origin rpy="0 0 0" xyz="0 0 0"/>
       </geometry>
@@ -82,5 +82,5 @@
     <visual>
       <geometry>
-        <mesh filename="file://$(find higgs2)/src/meshes/sonar_delantero.stl"/>
+        <mesh filename="file://$(find higgs2)/model/meshes/sonar_delantero.stl"/>
       </geometry>
       <origin rpy="0 0 0" xyz="0 0 0"/>
@@ -89,5 +89,5 @@
     <collision>
       <geometry>
-        <mesh filename="file://$(find higgs2)/src/meshes/sonar_delantero.stl"/>
+        <mesh filename="file://$(find higgs2)/model/meshes/sonar_delantero.stl"/>
         <sphere radius="0.01"/> <!-- <cylinder length="0.075" radius="0.111"/> -->
       </geometry>
@@ -105,5 +105,5 @@
     <visual>
       <geometry>
-        <mesh filename="file://$(find higgs2)/src/meshes/sonar_trasero.stl"/>
+        <mesh filename="file://$(find higgs2)/model/meshes/sonar_trasero.stl"/>
       </geometry>
       <origin rpy="0 0 0" xyz="0 0 0"/>
@@ -112,5 +112,5 @@
     <collision>
       <geometry>
-        <mesh filename="file://$(find higgs2)/src/meshes/sonar_trasero.stl"/>
+        <mesh filename="file://$(find higgs2)/model/meshes/sonar_trasero.stl"/>
       </geometry>
       <origin rpy="0 0 0" xyz="0 0 0"/>
@@ -144,12 +144,12 @@
       <origin rpy="0 0 0" xyz="0 0 0"/>
       <geometry>
-        <mesh filename="file://$(find higgs2)/src/meshes/eje.stl"/>
-      </geometry>
-      <material name="black"/>
-    </visual>
-    <collision>
-      <origin rpy="0 0 0" xyz="0 0 0"/>
-      <geometry>
-        <mesh filename="file://$(find higgs2)/src/meshes/eje.stl"/>
+        <mesh filename="file://$(find higgs2)/model/meshes/eje.stl"/>
+      </geometry>
+      <material name="black"/>
+    </visual>
+    <collision>
+      <origin rpy="0 0 0" xyz="0 0 0"/>
+      <geometry>
+        <mesh filename="file://$(find higgs2)/model/meshes/eje.stl"/>
       </geometry>
     </collision>
@@ -169,5 +169,5 @@
       <origin rpy="0 0 0" xyz="0 0 0"/>
       <geometry>
-        <mesh filename="file://$(find higgs2)/src/meshes/rueda.stl"/>
+        <mesh filename="file://$(find higgs2)/model/meshes/rueda.stl"/>
       </geometry>
       <material name="black"/>
@@ -209,12 +209,12 @@
       <origin rpy="0 0 0" xyz="0 0 0"/>
       <geometry>
-        <mesh filename="file://$(find higgs2)/src/meshes/eje.stl"/>
-      </geometry>
-      <material name="black"/>
-    </visual>
-    <collision>
-      <origin rpy="0 0 0" xyz="0 0 0"/>
-      <geometry>
-        <mesh filename="file://$(find higgs2)/src/meshes/eje.stl"/>
+        <mesh filename="file://$(find higgs2)/model/meshes/eje.stl"/>
+      </geometry>
+      <material name="black"/>
+    </visual>
+    <collision>
+      <origin rpy="0 0 0" xyz="0 0 0"/>
+      <geometry>
+        <mesh filename="file://$(find higgs2)/model/meshes/eje.stl"/>
       </geometry>
     </collision>
@@ -234,5 +234,5 @@
       <origin rpy="0 0 0" xyz="0 0 0"/>
       <geometry>
-        <mesh filename="file://$(find higgs2)/src/meshes/rueda.stl"/>
+        <mesh filename="file://$(find higgs2)/model/meshes/rueda.stl"/>
       </geometry>
       <material name="black"/>
@@ -274,12 +274,12 @@
       <origin rpy="0 0 0" xyz="0 0 0"/>
       <geometry>
-        <mesh filename="file://$(find higgs2)/src/meshes/eje.stl"/>
-      </geometry>
-      <material name="black"/>
-    </visual>
-    <collision>
-      <origin rpy="0 0 0" xyz="0 0 0"/>
-      <geometry>
-        <mesh filename="file://$(find higgs2)/src/meshes/eje.stl"/>
+        <mesh filename="file://$(find higgs2)/model/meshes/eje.stl"/>
+      </geometry>
+      <material name="black"/>
+    </visual>
+    <collision>
+      <origin rpy="0 0 0" xyz="0 0 0"/>
+      <geometry>
+        <mesh filename="file://$(find higgs2)/model/meshes/eje.stl"/>
       </geometry>
     </collision>
@@ -299,5 +299,5 @@
       <origin rpy="0 0 0" xyz="0 0 0"/>
       <geometry>
-        <mesh filename="file://$(find higgs2)/src/meshes/rueda.stl"/>
+        <mesh filename="file://$(find higgs2)/model/meshes/rueda.stl"/>
       </geometry>
       <material name="black"/>
@@ -339,12 +339,12 @@
       <origin rpy="0 0 0" xyz="0 0 0"/>
       <geometry>
-        <mesh filename="file://$(find higgs2)/src/meshes/eje.stl"/>
-      </geometry>
-      <material name="black"/>
-    </visual>
-    <collision>
-      <origin rpy="0 0 0" xyz="0 0 0"/>
-      <geometry>
-        <mesh filename="file://$(find higgs2)/src/meshes/eje.stl"/>
+        <mesh filename="file://$(find higgs2)/model/meshes/eje.stl"/>
+      </geometry>
+      <material name="black"/>
+    </visual>
+    <collision>
+      <origin rpy="0 0 0" xyz="0 0 0"/>
+      <geometry>
+        <mesh filename="file://$(find higgs2)/model/meshes/eje.stl"/>
       </geometry>
     </collision>
@@ -364,5 +364,5 @@
       <origin rpy="0 0 0" xyz="0 0 0"/>
       <geometry>
-        <mesh filename="file://$(find higgs2)/src/meshes/rueda.stl"/>
+        <mesh filename="file://$(find higgs2)/model/meshes/rueda.stl"/>
       </geometry>
       <material name="black"/>
