Commit message: map test

File: model/description/camera.xacro (robot description, xacro)
@@ -4,5 +4,5 @@
  <!-- |                                    CAMERA                                       | -->
  <!-- =================================================================================== -->
-    <link name="d_435_camera">
+    <link name="camera_link">
       <inertial>
         <mass value="0.001" />
@@ -25,6 +25,12 @@
       <origin xyz="0.2 0 0.2" rpy="0 0 0" />
       <parent link="base_link" />
-      <child link="d_435_camera" />
+      <child link="camera_link" />
     </joint>
+    <joint name="camera_optical_joint" type="fixed">
+        <parent link="camera_link"/>
+        <child link="camera_link_optical"/>
+        <origin xyz="0 0 0" rpy="${-pi/2} 0 ${-pi/2}"/>
+    </joint>
+    <link name="camera_link_optical"></link>
   <!-- INCLUDE CAMERA-->
     <gazebo reference="d_435_camera">

File: model/description/lidar.xacro (robot description, xacro)
@@ -23,5 +23,5 @@
  <joint name="hokuyo_joint" type="fixed">
     <axis xyz="0 1 0" />
-    <origin xyz="0.136 0 0.309" rpy="0 0 0"/>
+    <origin xyz="0.05 0 0.309" rpy="0 0 0"/> <!--0.136 x-->
     <parent link="base_link"/>
     <child link="hokuyo_link"/>

Commit message: few changes and views

File: model/description/camera.xacro (robot description, xacro)
@@ -34,5 +34,5 @@
     <link name="camera_link_optical"></link>
   <!-- INCLUDE CAMERA-->
-    <gazebo reference="d_435_camera">
+    <gazebo reference="camera_link">
     <sensor name="rgbd_camera" type="rgbd_camera">
       <always_on>true</always_on>

File: model/description/lidar.xacro (robot description, xacro)
@@ -23,5 +23,5 @@
  <joint name="hokuyo_joint" type="fixed">
     <axis xyz="0 1 0" />
-    <origin xyz="0.05 0 0.309" rpy="0 0 0"/> <!--0.136 x-->
+    <origin xyz="-0.1 0 0.309" rpy="0 0 0"/> <!--0.136 x-->
     <parent link="base_link"/>
     <child link="hokuyo_link"/>
